File: kicad/mqtt-thermocouple.kicad_pcb (KiCad board)
At the start: 2 copper layers, 91.4 x 66 mm, 35 parts, among them J1 Barrel_Jack, Q1 2N7000, Q2 2N7000, U1 MCP9600-E_MX, U2 CD4060BM96, U3 MAX6951

Commit message: revision A
Routing:
- net GND: track 7.70 -> 27.0 mm, vias 0 -> 1
- net Net-(TC1-Pad2): track 15.7 -> 18.3 mm
Other:
- board text added: "REVISION A JULY 2021"
- board text removed: "REVISION B APRIL 2021"

Commit message: revB
Parts:
- added R10: 4.7k, Resistor_SMD:R_1206_3216Metric_Pad1.30x1.75mm_HandSolder, F.Cu at (84.3, 93.0)
- added R4: 4.7k, Resistor_SMD:R_1206_3216Metric_Pad1.30x1.75mm_HandSolder, F.Cu at (81.8, 93.0)
- added REF**: OSHW-Logo2_9.8x8mm_SilkScreen, Symbol:OSHW-Logo2_9.8x8mm_SilkScreen, B.Cu at (99.1, 96.5)
- C4: value 1n -> 1u
- C7: value C -> 20p
- R3: value R_US -> 100k
Connections:
- net /display/~CS~ renamed /display/~{CS}
- A1 pad 12: (no net) -> unconnected-(A1-Pad12)
- A1 pad 15: (no net) -> unconnected-(A1-Pad15)
- A1 pad 16: (no net) -> unconnected-(A1-Pad16)
- A1 pad 19: (no net) -> unconnected-(A1-Pad19)
- A1 pad 2: (no net) -> unconnected-(A1-Pad2)
- A1 pad 20: (no net) -> unconnected-(A1-Pad20)
- A1 pad 3: (no net) -> unconnected-(A1-Pad3)
- A1 pad 9: (no net) -> unconnected-(A1-Pad9)
- PS1 pad 4: (no net) -> unconnected-(PS1-Pad4)
- U1 pad 11: (no net) -> unconnected-(U1-Pad11)
- U1 pad 12: (no net) -> unconnected-(U1-Pad12)
- U1 pad 14: (no net) -> unconnected-(U1-Pad14)
- U1 pad 15: (no net) -> unconnected-(U1-Pad15)
- U1 pad 21: Net-(U1-Pad21) -> unconnected-(U1-Pad21)
- U1 pad 22: Net-(U1-Pad21) -> unconnected-(U1-Pad21)
- U1 pad 23: Net-(U1-Pad21) -> unconnected-(U1-Pad21)
- U1 pad 24: Net-(U1-Pad21) -> unconnected-(U1-Pad21)
- U1 pad 25: Net-(U1-Pad21) -> unconnected-(U1-Pad21)
- U1 pad 26: Net-(U1-Pad21) -> unconnected-(U1-Pad21)
- U1 pad 27: Net-(U1-Pad21) -> unconnected-(U1-Pad21)
- U1 pad 28: Net-(U1-Pad21) -> unconnected-(U1-Pad21)
- U1 pad 29: Net-(U1-Pad21) -> unconnected-(U1-Pad21)
- U1 pad 30: Net-(U1-Pad21) -> unconnected-(U1-Pad21)
- U2 pad 1: (no net) -> unconnected-(U2-Pad1)
- U2 pad 13: (no net) -> unconnected-(U2-Pad13)
- U2 pad 14: (no net) -> unconnected-(U2-Pad14)
- U2 pad 15: (no net) -> unconnected-(U2-Pad15)
- U2 pad 2: (no net) -> unconnected-(U2-Pad2)
- U2 pad 4: (no net) -> unconnected-(U2-Pad4)
- U2 pad 5: (no net) -> unconnected-(U2-Pad5)
- U2 pad 6: (no net) -> unconnected-(U2-Pad6)
- U2 pad 7: (no net) -> unconnected-(U2-Pad7)
Routing:
- net +3V3: track 111.4 -> 121.9 mm
- net SCL: track 79.1 -> 87.1 mm, vias 1 -> 2
- net SDA: track 76.1 -> 83.0 mm, vias 1 -> 2
- net (no net): track 1.90 -> 0.00 mm
- net GND: track 27.0 -> 25.4 mm
- net unconnected-(A1-Pad19): track 0.00 -> 0.63 mm
- net unconnected-(A1-Pad16): track 0.00 -> 0.63 mm
- net unconnected-(A1-Pad9): track 0.00 -> 0.63 mm
Other:
- net class Default removed
- net class data removed
- board text added: "REVISION B APRIL 2022"
- board text added: "https://github.com/ uw-madison-chem-shops/ mqtt-thermocouple"
- board text removed: "REVISION A JULY 2021"

Commit message: checkpoint
Parts:
- removed the REF** at (99.1, 96.5)
- added U4: MAX31855KASA, Package_SO:SOIC-8_3.9x4.9mm_P1.27mm, F.Cu at (81.3, 101.6)
- moved C1 18.6 mm to (74.4, 50.2)
- moved R10 11.6 mm to (94.5, 87.4)
- moved R4 11.6 mm to (91.9, 87.4)
- moved U1 10.9 mm to (86.4, 88.9)
- moved C3 3.59 mm to (65.1, 76.2)
- moved PS1 1.80 mm to (54.6, 72.4)
- moved C2 0.37 mm to (51.4, 62.1)
Connections:
- A1 pad 16: unconnected-(A1-Pad16) -> Net-(A1-Pad16)
- Q1 pad 1: Net-(A1-Pad14) -> Net-(A1-Pad16)
Routing:
- net Net-(A1-Pad16): track 0.00 -> 66.4 mm
- net Net-(A1-Pad14): track 65.8 -> 0.00 mm
- net +3V3: track 121.9 -> 95.2 mm, vias 3 -> 2
- net Net-(TC1-Pad2): track 18.3 -> 0.00 mm
- net SCL: track 87.1 -> 72.5 mm
- net GND: track 25.4 -> 12.2 mm
- net SDA: track 83.0 -> 70.2 mm
- net Net-(C1-Pad1): track 34.4 -> 26.1 mm
- net Net-(TC1-Pad1): track 6.67 -> 0.00 mm
- net +5V: track 56.5 -> 59.4 mm
- net unconnected-(A1-Pad16): track 0.63 -> 0.00 mm
